File: pcb/ethernet_port.kicad_sch (KiCad schematic)
At the start: 3 parts, among them J3 RJ-064-1

Commit message: wip
Parts:
- J3: value RJ-064-1 -> MJ88-B211-JRS3; footprint MegaCard5_footprints:RJ-064-1 -> MegaCard5_footprints:MJ88-B211-JRS3; symbol MegaCard5_schematic_symbols:RJ-064-1 -> MegaCard5_schematic_symbols:MJ88-B211-JRS3; LCSC PN C7205199 -> C2895614; LCSC URL https://www.lcsc.com/product-detail/Ethernet-Connectors-Modular-Connectors-RJ45-RJ11_FG-RJ-064-1_C7205199.html -> https://www.lcsc.com/product-detail/Ethernet-Connectors-Modular-Connectors-RJ45-RJ11_Heling-MJ88-B211-JRS3_C2895614.html
Changed lines of the file:
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@@
 	)
 	(symbol
-		(lib_id "MegaCard5_schematic_symbols:RJ-064-1")
+		(lib_id "MegaCard5_schematic_symbols:MJ88-B211-JRS3")
 		(at 68.58 55.88 0)
 		(mirror y)
@@
 			)
 		)
-		(property "Value" "RJ-064-1"
+		(property "Value" "MJ88-B211-JRS3"
 			(at 77.47 55.8799 0)
 			(effects
@@
 			)
 		)
-		(property "Footprint" "MegaCard5_footprints:RJ-064-1"
+		(property "Footprint" "MegaCard5_footprints:MJ88-B211-JRS3"
 			(at 68.58 83.82 0)
 			(effects
@@
 			)
 		)
-		(property "Description" "RJ45Receptacle SMD Ethernet Connectors / Modular Connectors (RJ45 RJ11) ROHS"
+		(property "Description" "RJ45Receptacle 1 Shielded Horizontal attachment Without LED -25℃~+70℃ SMD Ethernet Connectors / Modular Connectors (RJ45 RJ11) ROHS"
 			(at 68.58 78.74 0)
 			(effects
@@
 			)
 		)
-		(property "LCSC PN" "C7205199"
+		(property "LCSC PN" "C2895614"
 			(at 68.58 86.36 0)
 			(effects
@@
 			)
 		)
-		(property "LCSC URL" "https://www.lcsc.com/product-detail/Ethernet-Connectors-Modular-Connectors-RJ45-RJ11_FG-RJ-064-1_C7205199.html"
+		(property "LCSC URL" "https://www.lcsc.com/product-detail/Ethernet-Connectors-Modular-Connectors-RJ45-RJ11_Heling-MJ88-B211-JRS3_C2895614.html"
 			(at 68.58 81.28 0)
 			(effects
