File: pcb/megacard5_reference_design.kicad_sch (KiCad schematic)
At the start: 22 parts, among them J1 MegaCard 5, J10 SMTSO2545CTJ, J11 5V, J12 3V3, J13 SMTSO2545CTJ, J14 GND, J15 VCC, J17 GND, J18 GND, J2 Barrel_Jack_Switch, J8 ~{EXT_RESET}, J9 ~{POWER_OFF}, SW1 POWER_OFF, SW2 RESET

Commit message: wip
Parts:
- removed J11: 5V, MegaCard5_footprints:5005, symbol MegaCard5_schematic_symbols:5005_red
- removed J12: 3V3, MegaCard5_footprints:5005, symbol MegaCard5_schematic_symbols:5005_red
- removed J14, J17, J18: GND, MegaCard5_footprints:5006, symbol MegaCard5_schematic_symbols:5006_black
- removed J15: VCC, MegaCard5_footprints:5005, symbol MegaCard5_schematic_symbols:5005_red
- removed J8: ~{EXT_RESET}, MegaCard5_footprints:5007, symbol MegaCard5_schematic_symbols:5007_white
- removed J9: ~{POWER_OFF}, MegaCard5_footprints:5007, symbol MegaCard5_schematic_symbols:5007_white
- removed R6: 4.7k, Resistor_SMD:R_1206_3216Metric, symbol Device:R_Small
- added J9: X2016WRS-16-9TSW, MegaCard5_footprints:X2016WRS-16-9TSW, symbol MegaCard5_schematic_symbols:X2016WRS-16-9TSW
- added SW3: AFT, MegaCard5_footprints:SKRPACE010, symbol MegaCard5_schematic_symbols:SKRPACE010
- added TP1: ~{POWER_OFF}, MegaCard5_footprints:5019, symbol MegaCard5_schematic_symbols:TestPoint
- added TP2: VCC, MegaCard5_footprints:5019, symbol MegaCard5_schematic_symbols:TestPoint
- added TP3: 5V, MegaCard5_footprints:5019, symbol MegaCard5_schematic_symbols:TestPoint
- added TP4: 3V3, MegaCard5_footprints:5019, symbol MegaCard5_schematic_symbols:TestPoint
- added TP5, TP6, TP7: GND, MegaCard5_footprints:5019, symbol MegaCard5_schematic_symbols:TestPoint
- added TP9: ~{EXT_RESET}, MegaCard5_footprints:5019, symbol MegaCard5_schematic_symbols:TestPoint
- J1: LCSC PN (none) -> C428485; LCSC URL (none) -> https://www.lcsc.com/product-detail/Edgeboard-Connectors_TE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
- J2: value Barrel_Jack_Switch -> 7V to 50V input; footprint Connector_BarrelJack:BarrelJack_Horizontal -> MegaCard5_footprints:DC-005-5A-2.0-SMT; symbol Connector:Barrel_Jack_Switch -> MegaCard5_schematic_symbols:DC-005-5A-2.0-SMT; LCSC PN C381116 -> C319134; LCSC URL https://www.lcsc.com/product-detail/DC-Power-Connectors_XKB-Connection-DC-005-5A-2-0_C381116.html -> https://www.lcsc.com/product-detail/DC-Power-Connectors_XKB-Connection-DC-005-5A-2-0-SMT_C319134.html
- SW1: value POWER_OFF -> ~{POWER_OFF}; footprint MegaCard5_footprints:SW_PUSH_6mm_H5mm -> MegaCard5_footprints:SKRPACE010; symbol MegaCard5_schematic_symbols:SKHWAQA010 -> MegaCard5_schematic_symbols:SKRPACE010; LCSC PN C139772 -> C139797; LCSC URL https://www.lcsc.com/product-detail/Tactile-Switches_ALPSALPINE-SKHWAQA010_C139772.html -> https://www.lcsc.com/product-detail/Tactile-Switches_ALPSALPINE-SKRPACE010_C139797.html
- SW2: value RESET -> ~{EXT_RESET}; footprint MegaCard5_footprints:SW_PUSH_6mm_H5mm -> MegaCard5_footprints:SKRPACE010; symbol MegaCard5_schematic_symbols:SKHWAQA010 -> MegaCard5_schematic_symbols:SKRPACE010; LCSC PN C139772 -> C139797; LCSC URL https://www.lcsc.com/product-detail/Tactile-Switches_ALPSALPINE-SKHWAQA010_C139772.html -> https://www.lcsc.com/product-detail/Tactile-Switches_ALPSALPINE-SKRPACE010_C139797.html
Connections:
- net +3.3V: now also J9.4 (Pin_4), SW3.1, TP4.1
- net +5V: now also J9.3 (Pin_3), TP3.1
- net GND: now also SW1.1, SW2.1, J9.14 (Pin_14), J9.15 (Pin_15), J9.16 (Pin_16), J9.2 (Pin_2), J9.MP, TP5.1, TP6.1, TP7.1; no longer SW1.2, SW2.2
- net VCC: now also TP2.1
- net VIN: now also J9.1 (Pin_1)
- net ~{EXT_RESET}: now also SW2.2, J9.5 (Pin_5), TP9.1; no longer SW2.1
- net ~{POWER_OFF}: now also SW1.2, J9.6 (Pin_6), TP1.1
- net AFT: now reaches J1.10 (RESERVED)
- net AFT: now also J9.7 (Pin_7), SW3.2
- net SCL/MDC: now reaches J1.12 (SCL/MDC)
- net SCL/MDC: now also J9.8 (Pin_8)
- net SDA/MDIO: now reaches J1.14 (SDA/MDIO)
- net SDA/MDIO: now also J9.9 (Pin_9)
- net DBG_SWDIO: now reaches J1.17 (RESERVED)
- net DBG_SWDIO: now also J9.12 (Pin_12)
- net GPIO0: now reaches J1.18 (RESERVED)
- net GPIO0: now also J9.10 (Pin_10)
- net DBG_SWCLK: now reaches J1.19 (RESERVED)
- net DBG_SWCLK: now also J9.13 (Pin_13)
- net GPIO1: now reaches J1.20 (RESERVED)
- net GPIO1: now also J9.11 (Pin_11)
- no-connect marks 8 -> 1
Other:
- note added: "Optional AFT button"
- note added: "Optional DC jack"
- note added: "Optional debugging connector"
- note added: "Optional test hooks"
- note removed: "Power input to board"
- note removed: "Test hooks"
- moved on the sheet: H1, H2, H3, H4, SCREW1, SCREW2

Commit message: updated PCB to Rev 1.1
Parts:
- removed J9: X2016WRS-16-9TSW, MegaCard5_footprints:X2016WRS-16-9TSW, symbol MegaCard5_schematic_symbols:X2016WRS-16-9TSW
- added J11, J12: S7B-PH-SM4-TB(LF)(SN), MegaCard5_footprints:JST_PH_S7B-PH-SM4-TB_1x07-1MP_P2.00mm_Horizontal, symbol MegaCard5_schematic_symbols:S7B-PH-SM4-TB(LF)(SN)
- H1, H2, H3, H4: now in the parts list
Connections:
- net +3.3V: now also J11.4 (Pin_4)
- net +5V: now also J11.3 (Pin_3)
- net AFT: now also J11.7 (Pin_7)
- net DBG_SWCLK: now also J12.7 (Pin_7)
- net DBG_SWDIO: now also J12.6 (Pin_6)
- net GND: now also J11.2 (Pin_2), J11.MP, J12.1 (Pin_1), J12.MP
- net GPIO0: now also J12.4 (Pin_4)
- net GPIO1: now also J12.5 (Pin_5)
- net SCL/MDC: now also J12.2 (Pin_2)
- net SDA/MDIO: now also J12.3 (Pin_3)
- net VIN: now also J11.1 (Pin_1)
- net ~{EXT_RESET}: now also J11.5 (Pin_5)
- net ~{POWER_OFF}: now also J11.6 (Pin_6)
Other:
- note added: "Optional debugging connectors"
- note removed: "Optional debugging connector"
